File: PCB/LPC804_LED_test_board_rev_01/_saved_LPC804_LED_test_board_rev_01.sch (KiCad schematic (older format))
At the start: 16 parts, among them J1 Conn_02x05_Odd_Even, U1 L78L06_SOT89, U2 L78L33_SOT89, U3 LPC804-TSSOP24

Commit message: Generated Netlist
Parts:
- added Q1: PN2222A, Package_TO_SOT_THT:TO-92_Inline, symbol Transistor_BJT:PN2222A
- added RN1: R_Pack04, symbol Device:R_Pack04
- BT1, BT2, BT3: footprint (none) -> Battery:BatteryHolder_Keystone_1060_1x2032
- C1, C2, C3, C4, C5, C6: footprint (none) -> Capacitor_SMD:C_0805_2012Metric
- J1: footprint (none) -> Connector_PinHeader_1.27mm:PinHeader_2x05_P1.27mm_Vertical
- U3: footprint (none) -> Package_SO:TSSOP-24_4.4x7.8mm_P0.65mm
Connections:
- net 6v: now also RN1.8 (R1.2)
- net GND: now also Q1.1 (E)
- net WS_Data renamed R1
- net R1: now also Q1.3 (C), RN1.1 (R1.1); no longer U3.1 (PIO0_18)
- new net: RN1.2 (R2.1), RN1.3 (R3.1)
- new net: RN1.5 (R4.2), RN1.6 (R3.2)
- new net WS_Data_MCU: RN1.7 (R2.2), U3.1 (PIO0_18)
- new net trig: Q1.2 (B), RN1.4 (R4.1)
Changed lines of the file:
@@
 F 0 "C1" H 1178 1046 50  0000 L CNN
 F 1 "CAP" H 1178 955 50  0000 L CNN
-F 2 "" H 1000 1000 50  0001 C CNN
+F 2 "Capacitor_SMD:C_0805_2012Metric" H 1000 1000 50  0001 C CNN
 F 3 "~" H 1000 1000 50  0001 C CNN
 	1    1000 1000
@@
 F 0 "C3" H 2528 1046 50  0000 L CNN
 F 1 "CAP" H 2528 955 50  0000 L CNN
-F 2 "" H 2350 1000 50  0001 C CNN
+F 2 "Capacitor_SMD:C_0805_2012Metric" H 2350 1000 50  0001 C CNN
 F 3 "~" H 2350 1000 50  0001 C CNN
 	1    2350 1000
@@
 F 0 "C2" H 1178 1896 50  0000 L CNN
 F 1 "CAP" H 1178 1805 50  0000 L CNN
-F 2 "" H 1000 1850 50  0001 C CNN
+F 2 "Capacitor_SMD:C_0805_2012Metric" H 1000 1850 50  0001 C CNN
 F 3 "~" H 1000 1850 50  0001 C CNN
 	1    1000 1850
@@
 F 0 "C4" H 2528 1896 50  0000 L CNN
 F 1 "CAP" H 2528 1805 50  0000 L CNN
-F 2 "" H 2350 1850 50  0001 C CNN
+F 2 "Capacitor_SMD:C_0805_2012Metric" H 2350 1850 50  0001 C CNN
 F 3 "~" H 2350 1850 50  0001 C CNN
 	1    2350 1850
@@
 F 0 "U3" H 2200 3978 50  0000 C CNN
 F 1 "LPC804-TSSOP24" H 2200 3887 50  0000 C CNN
-F 2 "" H 1500 3150 50  0001 C CNN
+F 2 "Package_SO:TSSOP-24_4.4x7.8mm_P0.65mm" H 1500 3150 50  0001 C CNN
 F 3 "" H 1500 3150 50  0001 C CNN
 	1    2200 3150
@@
 Wire Notes Line
 	6900 1600 6900 500
-Text GLabel 900  2700 0    50   Input ~ 0
-WS_Data
+Text GLabel 1050 2400 0    50   Input ~ 0
+WS_Data_MCU
 Wire Wire Line
 	900  2700 1000 2700
@@
 F 0 "J1" H 1200 4867 50  0000 C CNN
 F 1 "Conn_02x05_Odd_Even" H 1200 4776 50  0000 C CNN
-F 2 "" H 1150 4450 50  0001 C CNN
+F 2 "Connector_PinHeader_1.27mm:PinHeader_2x05_P1.27mm_Vertical" H 1150 4450 50  0001 C CNN
 F 3 "~" H 1150 4450 50  0001 C CNN
 	1    1150 4450
@@
 F 0 "C5" H 2878 4346 50  0000 L CNN
 F 1 "CAP" H 2878 4255 50  0000 L CNN
-F 2 "" H 2700 4300 50  0001 C CNN
+F 2 "Capacitor_SMD:C_0805_2012Metric" H 2700 4300 50  0001 C CNN
 F 3 "~" H 2700 4300 50  0001 C CNN
 	1    2700 4300
@@
 F 0 "C6" H 3378 4346 50  0000 L CNN
 F 1 "CAP" H 3378 4255 50  0000 L CNN
-F 2 "" H 3200 4300 50  0001 C CNN
+F 2 "Capacitor_SMD:C_0805_2012Metric" H 3200 4300 50  0001 C CNN
 F 3 "~" H 3200 4300 50  0001 C CNN
 	1    3200 4300
@@
 F 0 "BT1" H 4318 2146 50  0000 L CNN
 F 1 "Battery_Cell" H 4318 2055 50  0000 L CNN
-F 2 "" V 4200 2110 50  0001 C CNN
+F 2 "Battery:BatteryHolder_Keystone_1060_1x2032" V 4200 2110 50  0001 C CNN
 F 3 "~" V 4200 2110 50  0001 C CNN
 	1    4200 2050
@@
 F 0 "BT3" H 4318 3146 50  0000 L CNN
 F 1 "Battery_Cell" H 4318 3055 50  0000 L CNN
-F 2 "" V 4200 3110 50  0001 C CNN
+F 2 "Battery:BatteryHolder_Keystone_1060_1x2032" V 4200 3110 50  0001 C CNN
 F 3 "~" V 4200 3110 50  0001 C CNN
 	1    4200 3050
@@
 F 0 "BT2" H 4318 2596 50  0000 L CNN
 F 1 "Battery_Cell" H 4318 2505 50  0000 L CNN
-F 2 "" V 4200 2560 50  0001 C CNN
+F 2 "Battery:BatteryHolder_Keystone_1060_1x2032" V 4200 2560 50  0001 C CNN
 F 3 "~" V 4200 2560 50  0001 C CNN
 	1    4200 2500
@@
 Wire Notes Line
 	4850 3550 4850 1600
+$Comp
+L Transistor_BJT:PN2222A Q1
+U 1 1 5DB9156E
+P 5700 2250
+F 0 "Q1" H 5891 2296 50  0000 L CNN
+F 1 "PN2222A" H 5891 2205 50  0000 L CNN
+F 2 "Package_TO_SOT_THT:TO-92_Inline" H 5900 2175 50  0001 L CIN
+F 3 "http://www.fairchildsemi.com/ds/PN/PN2222A.pdf" H 5700 2250 50  0001 L CNN
+	1    5700 2250
+	1    0    0    -1
+$EndComp
+$Comp
+L Device:R_Pack04 RN1
+U 1 1 5DB91ECF
+P 6600 2250
+F 0 "RN1" H 6788 2296 50  0000 L CNN
+F 1 "R_Pack04" H 6788 2205 50  0000 L CNN
+F 2 "" V 6875 2250 50  0001 C CNN
+F 3 "~" H 6600 2250 50  0001 C CNN
+	1    6600 2250
+	1    0    0    -1
+$EndComp
+$Comp
+L power:GND #PWR010
+U 1 1 5DB920B1
+P 5800 2600
+F 0 "#PWR010" H 5800 2350 50  0001 C CNN
+F 1 "GND" H 5805 2427 50  0000 C CNN
+F 2 "" H 5800 2600 50  0001 C CNN
+F 3 "" H 5800 2600 50  0001 C CNN
+	1    5800 2600
+	1    0    0    -1
+$EndComp
+Wire Wire Line
+	5800 2450 5800 2600
+Text GLabel 5750 1900 0    50   Input ~ 0
+R1
+Wire Wire Line
+	5750 1900 5800 1900
+Wire Wire Line
+	5800 1900 5800 2050
+Text GLabel 6300 2550 0    50   Input ~ 0
+R1
+Wire Wire Line
+	6400 2450 6400 2550
+Wire Wire Line
+	6400 2550 6300 2550
+Text GLabel 6300 1850 0    50   Input ~ 0
+6v
+Wire Wire Line
+	6300 1850 6400 1850
+Wire Wire Line
+	6400 1850 6400 2050
+Wire Wire Line
+	6500 2450 6500 2550
+Wire Wire Line
+	6500 2550 6600 2550
+Wire Wire Line
+	6600 2550 6600 2450
+Wire Wire Line
+	6600 2050 6600 1950
+Wire Wire Line
+	6600 1950 6700 1950
+Wire Wire Line
+	6700 1950 6700 2050
+Text GLabel 6600 1850 2    50   Input ~ 0
+WS_Data_MCU
+Wire Wire Line
+	6600 1850 6500 1850
+Wire Wire Line
+	6500 1850 6500 2050
+Text GLabel 5300 2250 0    50   Input ~ 0
+trig
+Text GLabel 6750 2550 2    50   Input ~ 0
+trig
+Wire Wire Line
+	6750 2550 6700 2550
+Wire Wire Line
+	6700 2550 6700 2450
+Wire Wire Line
+	5300 2250 5500 2250
+Wire Wire Line
+	900  2700 900  2500
+Wire Wire Line
+	900  2500 1100 2500
+Wire Wire Line
+	1100 2500 1100 2400
+Wire Wire Line
+	1100 2400 1050 2400
+Text GLabel 6400 2800 0    50   Input ~ 0
+WS_Data
+Wire Wire Line
+	6400 2550 6400 2800
+Connection ~ 6400 2550
 $EndSCHEMATC
